File: Hardware/SparkFun_OpAmp_Breakout-LMV358.sch (EAGLE design)
At the start: 17 parts, among them IC1 LMV358

Commit message: Adding version number to schematic
Other:
- note added: "V16"
Changed lines of the file:
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@@
 <plain>
 <text x="101.6" y="68.58" size="2.54" layer="94" ratio="15">Av = (R1/R2)*(R4/R5) = 100</text>
+<text x="238.76" y="7.62" size="1.778" layer="94">V16</text>
 </plain>
 <instances>
